Commit message: Исправлена ошибка

File: src/go1_description/xacro/ros2_control.xacro (robot description, xacro)
@@ -2,7 +2,7 @@
 <robot xmlns:xacro="http://www.ros.org/wiki/xacro">
     <!-- <xacro:macro name="leg" params="name mirror mirror_dae front_hind front_hind_dae"> -->
-    <ros2_control name="GazeboSystem" type="system">
+    <ros2_control name="GazeboSimSystem" type="system">
         <hardware>
-            <plugin>gazebo_ros2_control/GazeboSystem</plugin>
+            <plugin>gz_ros2_control/GazeboSimSystem</plugin>
         </hardware>
         <joint name="FR_hip_joint">
@@ -317,8 +317,5 @@
     <!-- Gazebo's ros2_control plugin  -->
     <gazebo>
-        <plugin name="gazebo_ros2_control" filename="libgazebo_ros2_control.so">
-            <robot_sim_type>gazebo_ros2_control/GazeboSystem</robot_sim_type>
-            <robot_param>robot_description</robot_param>
-            <robot_param_node>robot_state_publisher_node</robot_param_node>
+        <plugin filename="libgz_ros2_control-system.so" name="gz_ros2_control::GazeboSimROS2ControlPlugin">
             <parameters>$(find go1_description)/config/jtc.yaml</parameters>
         </plugin>

File: src/go2_description/xacro/ros2_control.xacro (robot description, xacro)
@@ -2,7 +2,7 @@
 <robot xmlns:xacro="http://www.ros.org/wiki/xacro">
     <!-- <xacro:macro name="leg" params="name mirror mirror_dae front_hind front_hind_dae"> -->
-    <ros2_control name="GazeboSystem" type="system">
+    <ros2_control name="GazeboSimSystem" type="system">
         <hardware>
-            <plugin>gazebo_ros2_control/GazeboSystem</plugin>
+            <plugin>gz_ros2_control/GazeboSimSystem</plugin>
         </hardware>
         <joint name="FR_hip_joint">
@@ -114,211 +114,9 @@
             <state_interface name="effort" />
         </joint>
-        <!-- <joint name="FR_hip_joint">
-            <command_interface name="position">
-                <param name="min">${hip_position_min}</param>
-                <param name="max">${hip_position_max}</param>
-            </command_interface>
-            <command_interface name="velocity">
-                <param name="min">${hip_velocity_min}</param>
-                <param name="max">${hip_velocity_max}</param>
-            </command_interface>
-            <command_interface name="effort">
-                <param name="min">${hip_torque_min}</param>
-                <param name="max">${hip_torque_max}</param>
-            </command_interface>
-            <state_interface name="position"/>
-            <state_interface name="velocity"/>
-            <state_interface name="effort"/>
-        </joint>
-        <joint name="FR_thigh_joint">
-            <command_interface name="position">
-                <param name="min">${thigh_position_min}</param>
-                <param name="max">${thigh_position_max}</param>
-            </command_interface>
-            <command_interface name="velocity">
-                <param name="min">${thigh_velocity_min}</param>
-                <param name="max">${thigh_velocity_max}</param>
-            </command_interface>
-            <command_interface name="effort">
-                <param name="min">${thigh_torque_min}</param>
-                <param name="max">${thigh_torque_max}</param>
-            </command_interface>
-            <state_interface name="position"/>
-            <state_interface name="velocity"/>
-            <state_interface name="effort"/>
-        </joint>
-        <joint name="FR_calf_joint">
-            <command_interface name="position">
-                <param name="min">${calf_position_min}</param>
-                <param name="max">${calf_position_max}</param>
-            </command_interface>
-            <command_interface name="velocity">
-                <param name="min">${calf_velocity_min}</param>
-                <param name="max">${calf_velocity_max}</param>
-            </command_interface>
-            <command_interface name="effort">
-                <param name="min">${calf_torque_min}</param>
-                <param name="max">${calf_torque_max}</param>
-            </command_interface>
-            <state_interface name="position"/>
-            <state_interface name="velocity"/>
-            <state_interface name="effort"/>
-        </joint>
-        <joint name="FL_hip_joint">
-            <command_interface name="position">
-                <param name="min">${hip_position_min}</param>
-                <param name="max">${hip_position_max}</param>
-            </command_interface>
-            <command_interface name="velocity">
-                <param name="min">${hip_velocity_min}</param>
-                <param name="max">${hip_velocity_max}</param>
-            </command_interface>
-            <command_interface name="effort">
-                <param name="min">${hip_torque_min}</param>
-                <param name="max">${hip_torque_max}</param>
-            </command_interface>
-            <state_interface name="position"/>
-            <state_interface name="velocity"/>
-            <state_interface name="effort"/>
-        </joint>
-        <joint name="FL_thigh_joint">
-            <command_interface name="position">
-                <param name="min">${thigh_position_min}</param>
-                <param name="max">${thigh_position_max}</param>
-            </command_interface>
-            <command_interface name="velocity">
-                <param name="min">${thigh_velocity_min}</param>
-                <param name="max">${thigh_velocity_max}</param>
-            </command_interface>
-            <command_interface name="effort">
-                <param name="min">${thigh_torque_min}</param>
-                <param name="max">${thigh_torque_max}</param>
-            </command_interface>
-            <state_interface name="position"/>
-            <state_interface name="velocity"/>
-            <state_interface name="effort"/>
-        </joint>
-        <joint name="FL_calf_joint">
-            <command_interface name="position">
-                <param name="min">${calf_position_min}</param>
-                <param name="max">${calf_position_max}</param>
-            </command_interface>
-            <command_interface name="velocity">
-                <param name="min">${calf_velocity_min}</param>
-                <param name="max">${calf_velocity_max}</param>
-            </command_interface>
-            <command_interface name="effort">
-                <param name="min">${calf_torque_min}</param>
-                <param name="max">${calf_torque_max}</param>
-            </command_interface>
-            <state_interface name="position"/>
-            <state_interface name="velocity"/>
-            <state_interface name="effort"/>
-        </joint>
-        <joint name="RR_hip_joint">
-            <command_interface name="position">
-                <param name="min">${hip_position_min}</param>
-                <param name="max">${hip_position_max}</param>
-            </command_interface>
-            <command_interface name="velocity">
-                <param name="min">${hip_velocity_min}</param>
-                <param name="max">${hip_velocity_max}</param>
-            </command_interface>
-            <command_interface name="effort">
-                <param name="min">${hip_torque_min}</param>
-                <param name="max">${hip_torque_max}</param>
-            </command_interface>
-            <state_interface name="position"/>
-            <state_interface name="velocity"/>
-            <state_interface name="effort"/>
-        </joint>
-        <joint name="RR_thigh_joint">
-            <command_interface name="position">
-                <param name="min">${thigh_position_min}</param>
-                <param name="max">${thigh_position_max}</param>
-            </command_interface>
-            <command_interface name="velocity">
-                <param name="min">${thigh_velocity_min}</param>
-                <param name="max">${thigh_velocity_max}</param>
-            </command_interface>
-            <command_interface name="effort">
-                <param name="min">${thigh_torque_min}</param>
-                <param name="max">${thigh_torque_max}</param>
-            </command_interface>
-            <state_interface name="position"/>
-            <state_interface name="velocity"/>
-            <state_interface name="effort"/>
-        </joint>
-        <joint name="RR_calf_joint">
-            <command_interface name="position">
-                <param name="min">${calf_position_min}</param>
-                <param name="max">${calf_position_max}</param>
-            </command_interface>
-            <command_interface name="velocity">
-                <param name="min">${calf_velocity_min}</param>
-                <param name="max">${calf_velocity_max}</param>
-            </command_interface>
-            <command_interface name="effort">
-                <param name="min">${calf_torque_min}</param>
-                <param name="max">${calf_torque_max}</param>
-            </command_interface>
-            <state_interface name="position"/>
-            <state_interface name="velocity"/>
-            <state_interface name="effort"/>
-        </joint>    -->
-        <!-- <joint name="RL_thigh_joint">
-            <command_interface name="position">
-                <param name="min">${thigh_position_min}</param>
-                <param name="max">${thigh_position_max}</param>
-            </command_interface>
-            <command_interface name="velocity">
-                <param name="min">${thigh_velocity_min}</param>
-                <param name="max">${thigh_velocity_max}</param>
-            </command_interface>
-            <command_interface name="effort">
-                <param name="min">${thigh_torque_min}</param>
-                <param name="max">${thigh_torque_max}</param>
-            </command_interface>
-            <state_interface name="position"/>
-            <state_interface name="velocity"/>
-            <state_interface name="effort"/>
-        </joint>
-        <joint name="RL_calf_joint">
-            <command_interface name="position">
-                <param name="min">${calf_position_min}</param>
-                <param name="max">${calf_position_max}</param>
-            </command_interface>
-            <command_interface name="velocity">
-                <param name="min">${calf_velocity_min}</param>
-                <param name="max">${calf_velocity_max}</param>
-            </command_interface>
-            <command_interface name="effort">
-                <param name="min">${calf_torque_min}</param>
-                <param name="max">${calf_torque_max}</param>
-            </command_interface>
-            <state_interface name="position"/>
-            <state_interface name="velocity"/>
-            <state_interface name="effort"/>
-        </joint>      -->
-        <!-- <sensor name="imu_sensor">
-            <state_interface name="orientation.x"/>
-            <state_interface name="orientation.y"/>
-            <state_interface name="orientation.z"/>
-            <state_interface name="angular_velocity.x"/>
-            <state_interface name="angular_velocity.y"/>
-            <state_interface name="angular_velocity.z"/>
-            <state_interface name="linear_acceleration.x"/>
-            <state_interface name="linear_acceleration.y"/>
-            <state_interface name="linear_acceleration.z"/>
-            <param name="frame_id">imu_link</param>
-        </sensor> -->
     </ros2_control>
     <!-- </xacro:macro> -->
     <!-- Gazebo's ros2_control plugin  -->
     <gazebo>
-        <plugin name="gazebo_ros2_control" filename="libgazebo_ros2_control.so">
-            <robot_sim_type>gazebo_ros2_control/GazeboSystem</robot_sim_type>
-            <robot_param>robot_description</robot_param>
-            <robot_param_node>robot_state_publisher_node</robot_param_node>
+        <plugin filename="libgz_ros2_control-system.so" name="gz_ros2_control::GazeboSimROS2ControlPlugin">
             <parameters>$(find go2_description)/config/jtc.yaml</parameters>
         </plugin>
