Commit message: Миграция на Gazebo Harmonic и ROS2 Jazzy

File: src/go2_description/xacro/gazebo.xacro (robot description, xacro)
@@ -1,38 +1,11 @@
 <?xml version="1.0"?>
-<robot>
-    <!-- ros_control plugin -->
-    <!-- <gazebo>
-        <plugin name="gazebo_ros_control" filename="libgazebo_ros_control.so">
-            <robotNamespace>/go2_gazebo</robotNamespace>
-            <robotSimType>gazebo_ros_control/DefaultRobotHWSim</robotSimType>
-        </plugin>
-    </gazebo> -->
-    <!-- Show the trajectory of trunk center. -->
-    <!--gazebo>
-        <plugin name="3dplot" filename="libLinkPlot3DPlugin.so">
-            <frequency>10</frequency>
-            <plot>
-                <link>base</link>
-                <pose>0 0 0 0 0 0</pose>
-                <material>Gazebo/Yellow</material>
-            </plot>
-        </plugin>
-    </gazebo-->
-    <!-- Show the trajectory of foot. You can add another trajectory about another foot. -->
-    <!-- <gazebo>
-        <plugin name="3dplot" filename="libLinkPlot3DPlugin.so">
-            <frequency>100</frequency>
-            <plot>
-                <link>FL_foot</link>
-                <pose>0 0 0 0 0 0</pose>
-            </plot>
-        </plugin>
-    </gazebo>
-    <gazebo>
-        <plugin filename="libgazebo_ros_force.so" name="gazebo_ros_force">
-            <bodyName>trunk</bodyName>
-            <topicName>/apply_force/trunk</topicName>
-        </plugin>
-    </gazebo> -->
+<robot xmlns:xacro="http://ros.org/wiki/xacro">
+    <!--
+        Этот xacro подготовлен для миграции на Gazebo Harmonic (ros_gz).
+        По умолчанию `use_gazebo_classic` = false — плагины Gazebo Classic не включаются.
+        Если нужно запустить старый Gazebo Classic, передайте параметр xacro
+        `use_gazebo_classic:=true` при генерации/включении xacro.
+    -->
+    <xacro:property name="use_gazebo_classic" value="false"/>
     <gazebo reference="imu_link">
         <gravity>true</gravity>
@@ -42,13 +15,16 @@
             <visualize>true</visualize>
             <topic>__default_topic__</topic>
-            <plugin filename="libgazebo_ros_imu_sensor.so" name="imu_plugin">
-                <topicName>trunk_imu</topicName>
-                <bodyName>imu_link</bodyName>
-                <updateRateHZ>1000.0</updateRateHZ>
-                <gaussianNoise>0.0</gaussianNoise>
-                <xyzOffset>0 0 0</xyzOffset>
-                <rpyOffset>0 0 0</rpyOffset>
-                <frameName>imu_link</frameName>
-            </plugin>
+            <xacro:if value="${use_gazebo_classic}">
+                <plugin filename="libgazebo_ros_imu_sensor.so" name="imu_plugin">
+                    <topicName>trunk_imu</topicName>
+                    <bodyName>imu_link</bodyName>
+                    <updateRateHZ>1000.0</updateRateHZ>
+                    <gaussianNoise>0.0</gaussianNoise>
+                    <xyzOffset>0 0 0</xyzOffset>
+                    <rpyOffset>0 0 0</rpyOffset>
+                    <frameName>imu_link</frameName>
+                </plugin>
+            </xacro:if>
+            <!-- Для Gazebo Harmonic (ros_gz) используйте мост `ros_gz`/`parameter_bridge` для публикации IMU -->
             <pose>0 0 0 0 0 0</pose>
         </sensor>
@@ -58,5 +34,5 @@
         <sensor name="front_laser_sensor" type="ray">
             <always_on>true</always_on>
-            <visualize>false</visualize>            <!-- на Gazebo будет отображаться синие лучи -->
+            <visualize>false</visualize>
             <pose>0 0 0 0 0 0</pose>
             <update_rate>5</update_rate>
@@ -81,22 +57,28 @@
                 </noise>
             </ray>
-            <plugin name="gazebo_ros_front_laserscan" filename="libgazebo_ros_ray_sensor.so">
-                <ros>
-                    <remapping>~/out:=scan</remapping>
-                </ros>
-                <output_type>sensor_msgs/LaserScan</output_type>
-                <frame_name>front_laser</frame_name>
-            </plugin>
+            <xacro:if value="${use_gazebo_classic}">
+                <plugin name="gazebo_ros_front_laserscan" filename="libgazebo_ros_ray_sensor.so">
+                    <ros>
+                        <remapping>~/out:=scan</remapping>
+                    </ros>
+                    <output_type>sensor_msgs/LaserScan</output_type>
+                    <frame_name>front_laser</frame_name>
+                </plugin>
+            </xacro:if>
+            <!-- В Gazebo Harmonic: настройте ros_gz parameter_bridge для выдачи LaserScan -->
         </sensor>
     </gazebo>
-    <!-- Плагин одометрия -->
+    <!-- Плагин одометрия (classic) -->
     <gazebo>
-        <plugin name="p3d_ground_truth" filename="libgazebo_ros_p3d.so">
-            <!-- <robotNamespace>${g_robot_name}</robotNamespace> -->
-            <body_name>base_link</body_name>
-            <topic_name>odom</topic_name>
-            <frame_name>odom</frame_name>
-            <update_rate>100.0</update_rate>
-        </plugin>
+        <xacro:if value="${use_gazebo_classic}">
+            <plugin name="p3d_ground_truth" filename="libgazebo_ros_p3d.so">
+                <!-- <robotNamespace>${g_robot_name}</robotNamespace> -->
+                <body_name>base_link</body_name>
+                <topic_name>odom</topic_name>
+                <frame_name>odom</frame_name>
+                <update_rate>100.0</update_rate>
+            </plugin>
+        </xacro:if>
+        <!-- Для Harmonic используйте bridge/ros_gz для публикации одометрии / ground truth -->
     </gazebo>
     <gazebo reference="base_link">

Commit message: feat: синхронизировать FPS камеры и YOLO через update_rate gazebo.xacro
Цепочка: Makefile FPS -> camera_fps launch arg -> camera_fps xacro arg
-> <update_rate>${camera_fps}</update_rate>

Изменения:
- gazebo.xacro: camera_fps param макроса, дефолт 10
- robot.xacro: camera_fps xacro arg, проброс в gazebo macro
- Оба launch (py/cpp) мира: camera_fps launch arg + OpaqueFunction
- Оба launch (py/cpp) верхнего уровня: camera_fps launch arg, передача
  в мир через launch_arguments
- simulation.mk: make gazebo/gazebo-py/gazebo-cpp FPS=<N>
- Исправление: make gazebo теперь вызывает launch_python.launch.py
  (раньше несуществующий launch.launch.py)

File: src/go2_description/xacro/gazebo.xacro (robot description, xacro)
@@ -1,5 +1,5 @@
 <?xml version="1.0"?>
-<robot xmlns:xacro="http://www.ros.org/wiki/xacro" >
-    <xacro:macro  name="robot_gazebo_sensors" params="robot_name">
+<robot xmlns:xacro="http://www.ros.org/wiki/xacro">
+    <xacro:macro name="robot_gazebo_sensors" params="robot_name camera_fps:=10">
         <gazebo>
             <plugin name="gz_ros2_control::GazeboSimROS2ControlPlugin" filename="libgz_ros2_control-system.so">
@@ -96,8 +96,8 @@
                 <visualize>false</visualize>
                 <topic>/${robot_name}/imu_plugin/out</topic>
-                    <plugin filename="libgz-sim-imu-system.so" name="gz::sim::systems::Imu">
+                <plugin filename="libgz-sim-imu-system.so" name="gz::sim::systems::Imu">
                 </plugin>
                 <pose>0 0 0 0 0 0</pose>
-                <gz_frame_id>imu_link</gz_frame_id> <!-- Добавьте этот тег для указания кадра -->
+                <gz_frame_id>imu_link</gz_frame_id>                <!-- Добавьте этот тег для указания кадра -->
             </sensor>
         </gazebo>
@@ -130,5 +130,5 @@
                 <pose> 0 0 0 0 0 0 </pose>
                 <visualize>true</visualize>
-                <update_rate>30</update_rate>
+                <update_rate>${camera_fps}</update_rate>
                 <camera>
                     <camera_info_topic>/${robot_name}/color/camera_info</camera_info_topic>

File: src/go2_description/xacro/robot.xacro (robot description, xacro)
@@ -1,5 +1,7 @@
 <?xml version="1.0"?>
-<robot name="robot" xmlns:xacro="http://www.ros.org/wiki/xacro">
+<robot name="robot"
+    xmlns:xacro="http://www.ros.org/wiki/xacro">
     <xacro:arg name="DEBUG" default="false"/>
+    <xacro:arg name="camera_fps" default="10"/>
     <xacro:include filename="$(find go2_description)/xacro/const.xacro"/>
     <xacro:include filename="$(find go2_description)/xacro/materials.xacro"/>
@@ -8,5 +10,5 @@
     <xacro:include filename="$(find go2_description)/xacro/gazebo.xacro"/>
     <!-- <xacro:include filename="$(find go2_description)/launch/stairs.urdf.xacro"/> -->
-    <xacro:robot_gazebo_sensors robot_name="$(arg robot_name)"/>
+    <xacro:robot_gazebo_sensors robot_name="$(arg robot_name)" camera_fps="$(arg camera_fps)"/>
     <!-- <xacro:stairs stairs="15" xpos="0" ypos="0" zpos="0" /> -->
     <!-- Rotor related joint and link is only for demonstrate location. -->
@@ -51,12 +53,10 @@
             <origin rpy="0 0 0" xyz="${trunk_com_x} ${trunk_com_y} ${trunk_com_z}"/>
             <mass value="${trunk_mass}"/>
-            <inertia
-                ixx="${trunk_ixx}" ixy="${trunk_ixy}" ixz="${trunk_ixz}"
-                iyy="${trunk_iyy}" iyz="${trunk_iyz}"
-                izz="${trunk_izz}"/>
+            <inertia ixx="${trunk_ixx}" ixy="${trunk_ixy}" ixz="${trunk_ixz}" iyy="${trunk_iyy}" iyz="${trunk_iyz}" izz="${trunk_izz}"/>
         </inertial>
     </link>
     <joint name='laser_scan' type='fixed'>
-        <parent link="base_link"/>,
+        <parent link="base_link"/>
+,
         <child link="laser_frame"/>
         <origin xyz="0.22 0.0 0.095" rpy="0 0 0" />
@@ -182,7 +182,7 @@
         </collision>
     </link>
-    <xacro:leg name="rf" mirror="-1" mirror_dae= "False" front_hind="1"  front_hind_dae="True"  />
-    <xacro:leg name="lf" mirror="1"  mirror_dae="True"   front_hind="1"  front_hind_dae="True"  />
-    <xacro:leg name="rh" mirror="-1" mirror_dae="False"  front_hind="-1" front_hind_dae="False" />
-    <xacro:leg name="lh" mirror="1"  mirror_dae="True"   front_hind="-1" front_hind_dae="False" />
+    <xacro:leg name="rf" mirror="-1" mirror_dae= "False" front_hind="1" front_hind_dae="True" />
+    <xacro:leg name="lf" mirror="1" mirror_dae="True" front_hind="1" front_hind_dae="True" />
+    <xacro:leg name="rh" mirror="-1" mirror_dae="False" front_hind="-1" front_hind_dae="False" />
+    <xacro:leg name="lh" mirror="1" mirror_dae="True" front_hind="-1" front_hind_dae="False" />
 </robot>
