Commit message: fix(elevation): исправить контроллер ros2_control, meshes rviz и maps
leg.xacro:
- Удалён дублирующий ros2_control блок каждой ноги с неправильным
  плагином gazebo_ros2_control/GazeboSystem
- Все 12 joint уже объявлены в gazebo.xacro (gz_ros2_control/GazeboSimSystem)
- Дублирование вызывало 'Tried to insert StateInterface with already
  existing key' → контроллер не работал, TF odom не публиковался

compose.yml:
- AMENT_PREFIX_PATH в elevation-env для резолва package://go2_description
- Монтирование go2_description/go1_description в elevation-контейнер
- Создание symlink /root/ws/install/go2_description → /ws/install
  (RViz резолвит меши робота по пути из robot_description контейнера)
- Монтирование ./data/gazebo/maps → /root/ws/maps (SLAM-карты)

rviz (nav2_default_view, rviz_ns):
- Description Topic: /robot_description → /robot1/robot_description
  (модель робота не отображалась из-за namespace)

File: src/go2_description/xacro/leg.xacro (robot description, xacro)
@@ -143,24 +143,8 @@
             </inertial>
         </link>
-        <ros2_control name="${name}" type="system">
-            <hardware>
-                <plugin>gazebo_ros2_control/GazeboSystem</plugin>
-            </hardware>
-            <joint name="${name}_hip_joint">
-                <command_interface name="effort"/>
-                <state_interface name="position"/>
-                <state_interface name="velocity"/>
-            </joint>
-            <joint name="${name}_upper_leg_joint">
-                <command_interface name="effort"/>
-                <state_interface name="position"/>
-                <state_interface name="velocity"/>
-            </joint>
-            <joint name="${name}_lower_leg_joint">
-                <command_interface name="effort"/>
-                <state_interface name="position"/>
-                <state_interface name="velocity"/>
-            </joint>
-        </ros2_control>
+        <!-- ros2_control блок для каждой ноги УДАЛЁН — все 12 joint
+             объявлены в gazebo.xacro (${robot_name}_GazeboSystem).
+             Дублирование вызывало "Tried to insert StateInterface with
+             already existing key". -->
         <!-- <xacro:leg_transmission name="${name}"/> -->
     </xacro:macro>
